Commit message: update model add lidar

File: turtlebot_description/robots/kobuki_singlehexagon_sensor3dtof.urdf.xacro (robot description, xacro)
@@ -10,6 +10,8 @@
   <xacro:include filename="$(find turtlebot_description)/urdf/stacks/singlehexagon.urdf.xacro"/>
   <xacro:include filename="$(find turtlebot_description)/urdf/sensors/sensor3dtof.urdf.xacro"/>
+  <xacro:include filename="$(find turtlebot_description)/urdf/sensors/lidar.urdf.xacro"/>
   <xacro:kobuki/>
   <xacro:stack_hexagons parent="base_link"/>
   <xacro:sensor_3dtof parent="base_link"/>
+  <xacro:sensor_lidar parent="plate_bottom_link"/>
 </robot>

File: turtlebot_description/urdf/sensors/sensor3dtof.urdf.xacro (robot description, xacro)
@@ -22,5 +22,5 @@
       <child link="camera_link"/>
     </joint>
-      <link name="camera_link">
+    <link name="camera_link">
       <visual>
        <origin xyz="0 0 0" rpy="0 0 ${M_PI/2}"/>
@@ -47,18 +47,18 @@
          files. However, for Gazebo simulation we need them, so we add them here.
          (Hence, don't publish them additionally!) -->
-	<joint name="camera_depth_joint" type="fixed">
-	  <origin xyz="0 ${2 * -tof_cam_py} 0" rpy="0 0 0" />
-	  <parent link="camera_rgb_frame" />
-	  <child link="camera_depth_frame" />
-	</joint>
-	<link name="camera_depth_frame"/>
-	<joint name="camera_depth_optical_joint" type="fixed">
-	  <origin xyz="0 0 0" rpy="${-M_PI/2} 0 ${-M_PI/2}" />
-	  <parent link="camera_depth_frame" />
-	  <child link="camera_depth_optical_frame" />
-	</joint>
-	<link name="camera_depth_optical_frame"/>
-	<!-- Kinect sensor for simulation -->
-	<xacro:turtlebot_sim_3dsensor/>
+    <joint name="camera_depth_joint" type="fixed">
+      <origin xyz="0 ${2 * -tof_cam_py} 0" rpy="0 0 0" />
+      <parent link="camera_rgb_frame" />
+      <child link="camera_depth_frame" />
+    </joint>
+    <link name="camera_depth_frame"/>
+    <joint name="camera_depth_optical_joint" type="fixed">
+      <origin xyz="0 0 0" rpy="${-M_PI/2} 0 ${-M_PI/2}" />
+      <parent link="camera_depth_frame" />
+      <child link="camera_depth_optical_frame" />
+    </joint>
+    <link name="camera_depth_optical_frame"/>
+    <!-- Kinect sensor for simulation -->
+    <xacro:turtlebot_sim_3dsensor/>
   </xacro:macro>
 </robot>

File: turtlebot_description/urdf/turtlebot_gazebo.urdf.xacro (robot description, xacro)
@@ -1,4 +1,5 @@
 <?xml version="1.0"?>
-<robot name="turtlebot_gazebo" xmlns:xacro="http://ros.org/wiki/xacro">
+<robot name="turtlebot_gazebo"
+  xmlns:xacro="http://ros.org/wiki/xacro">
   <!-- Microsoft Kinect / ASUS Xtion PRO Live for simulation -->
   <xacro:macro name="turtlebot_sim_3dsensor">
@@ -40,3 +41,30 @@
     </gazebo>
   </xacro:macro>
+  <xacro:macro name="turtlebot_sim_lidar">
+    <gazebo reference="lidar_link">
+      <sensor type="ray" name="laser">
+        <always_on>true</always_on>
+        <update_rate>30</update_rate>
+        <ray>
+          <scan>
+            <horizontal>
+              <samples>360</samples>
+              <resolution>1</resolution>
+              <min_angle>-2.3562</min_angle>
+              <max_angle>2.3562</max_angle>
+            </horizontal>
+          </scan>
+          <range>
+            <min>0.10</min>
+            <max>5.0</max>
+            <resolution>0.01</resolution>
+          </range>
+        </ray>
+        <plugin name="turtlebot_lidar_controller" filename="libgazebo_ros_laser.so">
+          <topicName>/scan</topicName>
+          <frameName>lidar_link</frameName>
+        </plugin>
+      </sensor>
+    </gazebo>
+  </xacro:macro>
 </robot>

File: turtlebot_description/urdf/turtlebot_properties.urdf.xacro (robot description, xacro)
@@ -29,3 +29,7 @@
 	<xacro:property name="tof_cam_py" value="0.0" />
 	<xacro:property name="tof_cam_pz" value="0.080" />
+   <!-- lidar sensor position based on base_link -->
+  <xacro:property name="lidar_px" value="0.0" />
+	<xacro:property name="lidar_py" value="0.0" />
+	<xacro:property name="lidar_pz" value="0.010" />
 </robot>
