Commit message: adjust 3dtof sensor simulation

File: turtlebot_description/urdf/sensors/sensor3dtof.urdf.xacro (robot description, xacro)
@@ -59,6 +59,6 @@
     </joint>
     <link name="camera_depth_optical_frame"/>
-    <!-- Kinect sensor for simulation -->
-    <xacro:turtlebot_sim_3dsensor/>
+    <!-- 3dtof sensor for simulation -->
+    <xacro:turtlebot_sim_3dtof_sensor/>
   </xacro:macro>
 </robot>

File: turtlebot_description/urdf/turtlebot_gazebo.urdf.xacro (robot description, xacro)
@@ -41,4 +41,45 @@
     </gazebo>
   </xacro:macro>
+  <!-- 3dtof sensor for simulation -->
+  <xacro:macro name="turtlebot_sim_3dtof_sensor">
+    <gazebo reference="camera_link">
+      <sensor type="depth" name="camera">
+        <always_on>true</always_on>
+        <update_rate>30.0</update_rate>
+        <camera>
+          <horizontal_fov>${60.0*M_PI/180.0}</horizontal_fov>
+          <image>
+            <format>B8G8R8</format>
+            <width>320</width>
+            <height>240</height>
+          </image>
+          <clip>
+            <near>0.05</near>
+            <far>5</far>
+          </clip>
+        </camera>
+        <plugin name="tof_camera_controller" filename="libgazebo_ros_openni_kinect.so">
+          <cameraName>camera</cameraName>
+          <alwaysOn>true</alwaysOn>
+          <updateRate>30</updateRate>
+          <imageTopicName>rgb/image_raw</imageTopicName>
+          <depthImageTopicName>depth/image_raw</depthImageTopicName>
+          <pointCloudTopicName>depth/points</pointCloudTopicName>
+          <cameraInfoTopicName>rgb/camera_info</cameraInfoTopicName>
+          <depthImageCameraInfoTopicName>depth/camera_info</depthImageCameraInfoTopicName>
+          <frameName>camera_depth_optical_frame</frameName>
+          <baseline>0.1</baseline>
+          <distortion_k1>0.0</distortion_k1>
+          <distortion_k2>0.0</distortion_k2>
+          <distortion_k3>0.0</distortion_k3>
+          <distortion_t1>0.0</distortion_t1>
+          <distortion_t2>0.0</distortion_t2>
+          <!-- pointCloudCutoff and pointCloudCutoffMax is the minimum and maximum distance for points -->
+          <pointCloudCutoff>0.05</pointCloudCutoff>
+          <pointCloudCutoffMax>1.50</pointCloudCutoffMax>
+        </plugin>
+      </sensor>
+    </gazebo>
+  </xacro:macro>
   <xacro:macro name="turtlebot_sim_lidar">
     <gazebo reference="lidar_link">

Commit message: adjust laser scan range, 3d sensor collision attrs

File: turtlebot_description/urdf/sensors/sensor3dtof.urdf.xacro (robot description, xacro)
@@ -23,17 +23,17 @@
     </joint>
     <link name="camera_link">
-      <visual>
+      <!-- <visual>
        <origin xyz="0 0 0" rpy="0 0 ${M_PI/2}"/>
         <geometry>
         <box size="0.01 0.01 0.01" />
-         <!-- <mesh filename="package://turtlebot_description/meshes/sensors/kinect.dae"/> -->
+         <mesh filename="package://turtlebot_description/meshes/sensors/kinect.dae"/>
         </geometry>
-      </visual>
-  	  <collision>
+      </visual> -->
+  	  <!-- <collision>
         <origin xyz="0.0 0.0 0.0" rpy="0 0 0"/>
   	    <geometry>
   	      <box size="0.01 0.01 0.01"/>
   	    </geometry>
-  	  </collision>
+  	  </collision> -->
       <inertial>
         <mass value="0.564" />

File: turtlebot_description/urdf/turtlebot_gazebo.urdf.xacro (robot description, xacro)
@@ -86,4 +86,5 @@
       <sensor type="ray" name="laser">
         <always_on>true</always_on>
+        <visualize>false</visualize>
         <update_rate>30</update_rate>
         <ray>
@@ -92,6 +93,6 @@
               <samples>360</samples>
               <resolution>1</resolution>
-              <min_angle>-2.3562</min_angle>
-              <max_angle>2.3562</max_angle>
+              <min_angle>-3.14</min_angle>
+              <max_angle>3.14</max_angle>
             </horizontal>
           </scan>
@@ -101,4 +102,13 @@
             <resolution>0.01</resolution>
           </range>
+          <noise>
+            <type>gaussian</type>
+            <!-- Noise parameters based on published spec for Hokuyo laser
+                achieving "+-30mm" accuracy at range < 10m.  A mean of 0.0m and
+                stddev of 0.01m will put 99.7% of samples within 0.03m of the true
+                reading. -->
+            <mean>0.0</mean>
+            <stddev>0.01</stddev>
+        </noise>
         </ray>
         <plugin name="turtlebot_lidar_controller" filename="libgazebo_ros_laser.so">
