Commit message: change laser link in gazebo model

File: turtlebot_description/urdf/sensors/lidar.urdf.xacro (robot description, xacro)
@@ -8,7 +8,7 @@
       <origin xyz="${lidar_px} ${lidar_py} ${lidar_pz}" rpy="0 0 0"/>
       <parent link="${parent}"/>
-      <child link="lidar_link" />
+      <child link="laser_link" />
     </joint>
-    <link name="lidar_link">
+    <link name="laser_link">
       <visual>
         <origin xyz="0.0 0.0 0.0" rpy="0 0 0"/>

File: turtlebot_description/urdf/turtlebot_gazebo.urdf.xacro (robot description, xacro)
@@ -83,5 +83,5 @@
   </xacro:macro>
   <xacro:macro name="turtlebot_sim_lidar">
-    <gazebo reference="lidar_link">
+    <gazebo reference="laser_link">
       <sensor type="ray" name="laser">
         <always_on>true</always_on>
@@ -114,5 +114,5 @@
         <plugin name="turtlebot_lidar_controller" filename="libgazebo_ros_laser.so">
           <topicName>/scan</topicName>
-          <frameName>lidar_link</frameName>
+          <frameName>laser_link</frameName>
         </plugin>
       </sensor>

Commit message: adjust sensor param

File: turtlebot_description/urdf/sensors/lidar.urdf.xacro (robot description, xacro)
@@ -14,5 +14,5 @@
         <origin xyz="0.0 0.0 0.0" rpy="0 0 0"/>
         <geometry>
-          <box size="0.01 0.01 0.01"/>
+          <cylinder radius="0.043" length="0.0546" />
         </geometry>
       </visual>

File: turtlebot_description/urdf/turtlebot_properties.urdf.xacro (robot description, xacro)
@@ -28,8 +28,10 @@
   <xacro:property name="tof_cam_px" value="0.180" />
 	<xacro:property name="tof_cam_py" value="0.0" />
-	<xacro:property name="tof_cam_pz" value="0.080" />
-   <!-- lidar sensor position based on base_link -->
+  <!-- tof离地高度 -->
+	<xacro:property name="tof_cam_pz" value="0.047" />
+   <!-- lidar sensor position based on plate_bottom_link -->
   <xacro:property name="lidar_px" value="0.0" />
 	<xacro:property name="lidar_py" value="0.0" />
-	<xacro:property name="lidar_pz" value="0.010" />
+  <!-- lidar距离机器人顶部的高度 -->
+	<xacro:property name="lidar_pz" value="0.041" />
 </robot>
