Commit message: create own robot model

File: turtlebot_description/urdf/turtlebot_properties.urdf.xacro (robot description, xacro)
@@ -25,3 +25,7 @@
 	<xacro:property name="cam_op" value="0" />
 	<xacro:property name="cam_oy" value="0" />
+  <!-- 3dtof sensor position based on base_link -->
+  <xacro:property name="tof_cam_px" value="0.180" />
+	<xacro:property name="tof_cam_py" value="0.0" />
+	<xacro:property name="tof_cam_pz" value="0.080" />
 </robot>

Commit message: fix tof sensor urdf param

File: turtlebot_description/urdf/turtlebot_properties.urdf.xacro (robot description, xacro)
@@ -29,5 +29,6 @@
 	<xacro:property name="tof_cam_py" value="0.0" />
   <!-- tof离地高度 -->
-	<xacro:property name="tof_cam_pz" value="0.047" />
+  <!-- height: base_footprint (ground) -> base_link(0.0102m) -> tof(0.037m) -->
+	<xacro:property name="tof_cam_pz" value="0.037" />
    <!-- lidar sensor position based on plate_bottom_link -->
   <xacro:property name="lidar_px" value="0.0" />
